File: SOURCE_FILES/BIM_PCB/BUCK_REGULATOR_ADP2504ACPZ-R7.kicad_sch (KiCad schematic)
At the start: 11 parts, among them U7 ADP2504ACPZ-R7_3.3V_VERSION

Commit message: updates on schematic and complete layout
Parts:
- C36: footprint Capacitor_SMD:C_0603_1608Metric -> Capacitor_SMD:C_0402_1005Metric
Changed lines of the file:
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@@
       (effects (font (size 1.27 1.27)) (justify left))
     )
-    (property "Footprint" "Capacitor_SMD:C_0603_1608Metric" (at 177.8 92.71 0)
+    (property "Footprint" "Capacitor_SMD:C_0402_1005Metric" (at 177.8 92.71 0)
       (effects (font (size 1.27 1.27)) hide)
     )

Commit message: complete BIM Board
Parts:
- R41: value 1K -> 0R; now not fitted
- R42: now not fitted
Changed lines of the file:
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@@
   )
   (symbol (lib_id "Device:R_US") (at 166.37 88.9 0) (unit 1)
-    (in_bom yes) (on_board yes) (dnp no) (fields_autoplaced)
+    (in_bom yes) (on_board yes) (dnp yes) (fields_autoplaced)
     (property "Reference" "R41" (at 168.91 88.265 0)
       (effects (font (size 1.27 1.27)) (justify left))
     )
-    (property "Value" "1K" (at 168.91 90.805 0)
+    (property "Value" "0R" (at 168.91 90.805 0)
       (effects (font (size 1.27 1.27)) (justify left))
     )
@@
   )
   (symbol (lib_id "Device:R_US") (at 166.37 101.6 0) (unit 1)
-    (in_bom yes) (on_board yes) (dnp no) (fields_autoplaced)
+    (in_bom yes) (on_board yes) (dnp yes) (fields_autoplaced)
     (property "Reference" "R42" (at 168.91 100.965 0)
       (effects (font (size 1.27 1.27)) (justify left))
