File: SOURCE_FILES/BIM_PCB/SY8089_BUCK_CONVERTER.kicad_sch (KiCad schematic)
At the start: 13 parts, among them U7 SY8089AAAC

Commit message: updated step
Parts:
- C20: footprint Capacitor_SMD:C_0603_1608Metric -> Capacitor_SMD:C_0402_1005Metric
Changed lines of the file:
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@@
       (effects (font (size 1.27 1.27)) (justify left))
     )
-    (property "Footprint" "Capacitor_SMD:C_0603_1608Metric" (at 157.48 99.695 0)
+    (property "Footprint" "Capacitor_SMD:C_0402_1005Metric" (at 157.48 99.695 0)
       (effects (font (size 1.27 1.27)) hide)
     )

Commit message: xmas
Other:
- note added: "SIM MODULE POWER SUPPLY 3V3/2A"
- note removed: "SIM MODULE POWER SUPPLY 4.2V/2A"
Changed lines of the file:
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@@
     (stroke (width 0) (type default))
-  )
-  (text "SIM MODULE POWER SUPPLY 4.2V/2A " (at 115.57 72.39 0)
-    (effects (font (face "Algerian") (size 3 3) (thickness 0.6) bold) (justify left bottom))
   )
   (text "Eliminates High Freq\ninterference\nPlace close to SIM\nVBAT pins"
@@
     (effects (font (face "KiCad Font") (size 1.27 1.27)) (justify left bottom))
   )
+  (text "SIM MODULE POWER SUPPLY 3V3/2A " (at 120.015 65.405 0)
+    (effects (font (face "Algerian") (size 3 3) (thickness 0.6) bold) (justify left bottom))
+  )
   (text "3V3 OUTPUT" (at 218.44 92.075 0)

Commit message: completed project and all the prouction files
Parts:
- C19: footprint Capacitor_SMD:C_0603_1608Metric -> Capacitor_SMD:C_0402_1005Metric
Changed lines of the file:
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@@
       (effects (font (size 1.27 1.27)) (justify left))
     )
-    (property "Footprint" "Capacitor_SMD:C_0603_1608Metric" (at 108.585 103.505 0)
+    (property "Footprint" "Capacitor_SMD:C_0402_1005Metric" (at 108.585 103.505 0)
       (effects (font (size 1.27 1.27)) hide)
     )
