File: SOURCE_FILES/BIM_PCB/BIM_PCB.kicad_pcb (KiCad board)
At the start: 4 copper layers, 63.5 x 72.5 mm, 208 parts, among them J1 Conn_02x09_Counter_Clockwise, J2 nano_sim, J3 Conn_01x06, J4 Micro_SD_Card, Q1 SSM3J328R-HXY, Q2 SSM3J328R-HXY, Q3 IRLML0100TRPBF, Q4 2N7002, Q5 BSN20, Q6 BSN20, Q7 2N7002, Q8 2N7002, Q9 2N7002, SW1 reset, U1 STM32F103C8Tx, U10 TBU-CA065-200-WH, U11 SSP3485U, U12 TBU-CA065-200-WH, U13 ATA6561-GAQW-N, U14 WAS3157B, U15 MC74HC4052A, U16 SY8089AAAC, U17 XC6206PxxxMR, U18 TBU-CA065-200-WH, U19 SSP3485U, U2 PCF8523TK, U20 TBU-CA065-200-WH, U3 A9G_MODULE, U4 TBU-CA065-200-WH, U5 SSP3485U, U6 TBU-CA065-200-WH, U7 WAS3157B, U8 W25Q32JVSS, U9 ATA6561-GAQW-N, Y1 8MHz, Y2 32.678KHz, Y3 32.678KHz

Commit message: completed project
Parts:
- D-1: moved to B.Cu
- J1: footprint Connector_Molex:Molex_Mini-Fit_Jr_5569-18A2_2x09_P4.20mm_Horizontal -> MACHADA_footprints:conn_18pin_02x09_angled_MX23A18NF1
- moved AE1 34.2 mm to (90.5, 60.7), turned to -90 degrees
- moved HST_TXD1 29.8 mm to (62.5, 60.0)
- moved D3 26.8 mm to (86.8, 60.3), turned to -90 degrees
- moved L2 24.8 mm to (85.7, 60.3), turned to -90 degrees
- moved HST_RXD1 23.9 mm to (68.0, 60.0)
- moved D+1 17.8 mm to (70.5, 61.8)
- moved C19 17.6 mm to (64.2, 62.0)
- moved R29 17.6 mm to (65.2, 62.0)
- moved D-1 17.0 mm to (71.2, 61.8), turned to 180 degrees
- moved J1 13.4 mm to (46.9, 93.9), turned to -90 degrees
- moved C18 11.7 mm to (66.5, 62.0)
- moved R30 11.7 mm to (67.5, 62.0)
- moved G*** 6.53 mm to (76.9, 59.7)
- moved J4 4.40 mm to (87.1, 91.5), turned to 90 degrees
- moved D16 3.66 mm to (37.5, 116.2)
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Connections:
- net Net-(J2-I/O) renamed /A9G_GSM_GPRS_MODULE/i/o
- C21 pad 1: /A9G_GSM_GPRS_MODULE/TF_CARD_CONN/2V8 -> 2V8
- C22 pad 1: /A9G_GSM_GPRS_MODULE/TF_CARD_CONN/2V8 -> 2V8
- HST_RXD1 pad 1: Net-(U3-HST_RXD) -> Net-(U3-HST_TXD)
- HST_TXD1 pad 1: Net-(U3-HST_TXD) -> Net-(U3-HST_RXD)
- J4 pad 4: /A9G_GSM_GPRS_MODULE/TF_CARD_CONN/2V8 -> 2V8
- R40 pad 1: /A9G_GSM_GPRS_MODULE/TF_CARD_CONN/2V8 -> 2V8
- R41 pad 1: /A9G_GSM_GPRS_MODULE/TF_CARD_CONN/2V8 -> 2V8
- R42 pad 1: /A9G_GSM_GPRS_MODULE/TF_CARD_CONN/2V8 -> 2V8
- R45 pad 1: /A9G_GSM_GPRS_MODULE/TF_CARD_CONN/2V8 -> 2V8
- R46 pad 1: /A9G_GSM_GPRS_MODULE/TF_CARD_CONN/2V8 -> 2V8
- R47 pad 1: /A9G_GSM_GPRS_MODULE/TF_CARD_CONN/2V8 -> 2V8
- U3 pad 28: /A9G_GSM_GPRS_MODULE/Sim_CLK -> Net-(AE1-A)
- U3 pad 29: /A9G_GSM_GPRS_MODULE/V_Sim -> GND
- U3 pad 30: /A9G_GSM_GPRS_MODULE/Sim_DIO -> /A9G_GSM_GPRS_MODULE/GPS POSITION
- U3 pad 31: Net-(U3-HST_RXD) -> unconnected-(U3-IO30-Pad31)
- U3 pad 32: Net-(U3-HST_TXD) -> unconnected-(U3-IO25-Pad32)
- U3 pad 33: Net-(U3-USB_P) -> unconnected-(U3-MIC_N-Pad33)
- U3 pad 34: Net-(U3-USB_N) -> unconnected-(U3-MIC_P-Pad34)
- U3 pad 35: unconnected-(U3-MIC_P-Pad35) -> Net-(U3-USB_N)
- U3 pad 36: unconnected-(U3-MIC_N-Pad36) -> Net-(U3-USB_P)
- U3 pad 37: unconnected-(U3-IO25-Pad37) -> Net-(U3-HST_TXD)
- U3 pad 38: unconnected-(U3-IO30-Pad38) -> Net-(U3-HST_RXD)
- U3 pad 39: /A9G_GSM_GPRS_MODULE/GPS POSITION -> /A9G_GSM_GPRS_MODULE/Sim_DIO
- U3 pad 40: GND -> /A9G_GSM_GPRS_MODULE/V_Sim
- U3 pad 41: Net-(AE1-A) -> /A9G_GSM_GPRS_MODULE/Sim_CLK
- U3 pad 46: unconnected-(U3-GND-Pad46) -> GND
Routing:
- net 2V8: track 43.2 -> 102.2 mm, vias 5 -> 8
- net /A9G_GSM_GPRS_MODULE/TF_CARD_CONN/2V8: track 26.3 -> 0.00 mm, vias 1 -> 0
- net /A9G_GSM_GPRS_MODULE/TF_CARD_CONN/SD_D3: track 17.7 -> 41.8 mm, vias 1 -> 2
- net /A9G_GSM_GPRS_MODULE/TF_CARD_CONN/SD_CMD: track 12.3 -> 32.9 mm, vias 1 -> 2
- net /A9G_GSM_GPRS_MODULE/Sim_Restart: track 47.3 -> 67.5 mm
- net Net-(U3-HST_TXD): track 25.8 -> 6.05 mm, vias 2 -> 0
- net /A9G_GSM_GPRS_MODULE/TF_CARD_CONN/SD_D2: track 24.0 -> 41.5 mm
- net /A9G_GSM_GPRS_MODULE/TF_CARD_CONN/SD_CLK: track 13.8 -> 30.5 mm, vias 1 -> 2
- net Net-(U3-USB_P): track 19.6 -> 3.58 mm, vias 2 -> 0
- net /A9G_GSM_GPRS_MODULE/IO29: track 31.3 -> 47.2 mm, vias 0 -> 2
- net Net-(U3-USB_N): track 19.6 -> 3.81 mm, vias 2 -> 1
- net /A9G_GSM_GPRS_MODULE/TF_CARD_CONN/SD_D1: track 16.7 -> 32.4 mm, vias 1 -> 2
- net 4.2V_SIMPWR: track 45.6 -> 30.6 mm, vias 7 -> 5
- net /A9G_GSM_GPRS_MODULE/GPS_TXD: track 98.1 -> 83.2 mm, vias 5 -> 4
- net /swdio: track 110.5 -> 96.5 mm
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Other:
- board size 63.5 x 72.5 mm -> 58.5 x 72.5 mm

Commit message: completed project and all the prouction files
Parts:
- removed Q4, Q7, Q8, Q9: 2N7002, Package_TO_SOT_SMD:SOT-23
- removed R17, R18, R48, R49, R52, R54, R55: 10K, Resistor_SMD:R_0402_1005Metric
- removed R19, R50, R53, R56: 1K, Resistor_SMD:R_0402_1005Metric
- removed SIM_I2C_SCL1: SIM_I2C_SCL, brilliant-kicad-library:TestPoint_Pad_D0.9mm
- removed SIM_I2C_SDA1: SIM_I2C_SDA, brilliant-kicad-library:TestPoint_Pad_D0.9mm
- added AE3: Antenna_Shield, greencharge-footprints:UFL_COAX_CONN23370191, F.Cu at (86.3, 60.0)
- added C35: 100u, Capacitor_Tantalum_SMD:CP_EIA-3216-18_Kemet-A, B.Cu at (78.5, 79.7)
- added C36: 100u, Capacitor_Tantalum_SMD:CP_EIA-3216-18_Kemet-A, B.Cu at (76.2, 79.7)
- added FL1: SAFEB1G57KE0F00R15, Filter:Filter_1411-5_1.4x1.1mm, F.Cu at (84.8, 64.7)
- AE1: footprint greencharge-footprints:UFL_COAX_CONN23370191 -> Connector_Coaxial:SMA_Samtec_SMA-J-P-X-ST-EM1_EdgeMount
- C28: value 100u -> 0.1u; footprint Capacitor_Tantalum_SMD:CP_EIA-3216-18_Kemet-A -> Capacitor_SMD:C_0402_1005Metric
- D5, D6: footprint LED_SMD:LED_0603_1608Metric -> LED_SMD:LED_0402_1005Metric
- R51: value 10K -> 0R
- moved D3 33.0 mm to (55.7, 71.3), turned to 90 degrees
- moved C28 10.5 mm to (79.0, 70.0), turned to -90 degrees
- moved R51 10.4 mm to (57.3, 70.8), turned to 180 degrees
- moved J2 5.24 mm to (80.4, 72.6)
- moved L2 4.97 mm to (86.4, 65.2)
- moved AE1 4.30 mm to (92.1, 64.7), turned to 90 degrees
- moved D4 3.07 mm to (77.7, 73.6)
- moved C29 1.14 mm to (60.7, 67.3)
- moved D11 0.83 mm to (69.7, 79.4)
- moved D12 0.83 mm to (73.4, 79.4)
- moved D10 0.82 mm to (66.2, 79.4)
- moved R36 0.60 mm to (72.7, 60.0)
- moved U20 0.22 mm to (44.5, 121.0)
- moved J1 0.22 mm to (46.7, 94.0)
- moved U18 0.11 mm to (44.7, 116.0)
Connections:
- net /A9G_GSM_GPRS_MODULE/i/o renamed Net-(J2-I/O)
- C28 pad 1: 4.2V_SIMPWR -> GND
- C28 pad 2: GND -> /A9G_GSM_GPRS_MODULE/V_Sim
- D3 pad 2: Net-(AE1-A) -> Net-(AE2-A)
- L2 pad 1: GND -> Net-(AE1-A)
- L2 pad 2: Net-(AE1-A) -> 4.2V_SIMPWR
- R51 pad 1: 2V8 -> Net-(U3-GSM_RF)
- R51 pad 2: Net-(Q8-S) -> Net-(AE2-A)
- U3 pad 28: Net-(AE1-A) -> Net-(U3-GPS_RF)
- U3 pad 45: Net-(AE2-A) -> Net-(U3-GSM_RF)
- U3 pad 49: /A9G_GSM_GPRS_MODULE/MOSFET_LOGIC_LEVEL_TRANSLATOR7/LOW_SIDE_LOGIC_SIGNAL -> /A9G_GSM_GPRS_MODULE/GPS_RXD
- U3 pad 50: /A9G_GSM_GPRS_MODULE/MOSFET_LOGIC_LEVEL_TRANSLATOR6/LOW_SIDE_LOGIC_SIGNAL -> /A9G_GSM_GPRS_MODULE/GPS_TXD
- U3 pad 53: /A9G_GSM_GPRS_MODULE/MOSFET_LOGIC_LEVEL_TRANSLATOR8/LOW_SIDE_LOGIC_SIGNAL -> /STM32FC8T6_MCU/RX1
- U3 pad 54: /A9G_GSM_GPRS_MODULE/MOSFET_LOGIC_LEVEL_TRANSLATOR9/LOW_SIDE_LOGIC_SIGNAL -> /STM32FC8T6_MCU/TX1
Routing:
- net +3V3: track 182.7 -> 142.8 mm, vias 19 -> 13
- net 2V8: track 102.2 -> 62.8 mm, vias 8 -> 3
- net VIN: track 0.00 -> 31.1 mm
- net Net-(J1-Pin_4): track 34.9 -> 16.9 mm
- net /A9G_GSM_GPRS_MODULE/GPS_TXD: track 83.2 -> 66.4 mm
- net 4.2V_SIMPWR: track 30.6 -> 46.7 mm, vias 5 -> 9
- net /A9G_GSM_GPRS_MODULE/MOSFET_LOGIC_LEVEL_TRANSLATOR6/LOW_SIDE_LOGIC_SIGNAL: track 16.1 -> 0.00 mm
- net /SW0: track 98.2 -> 86.6 mm
- net /RS485_B: track 10.7 -> 21.5 mm
- net /A9G_GSM_GPRS_MODULE/MOSFET_LOGIC_LEVEL_TRANSLATOR7/LOW_SIDE_LOGIC_SIGNAL: track 10.3 -> 0.00 mm
- net /ECU_A: track 10.2 -> 19.4 mm
- net /DIS_A: track 33.0 -> 42.2 mm
- net /A9G_GSM_GPRS_MODULE/MOSFET_LOGIC_LEVEL_TRANSLATOR9/LOW_SIDE_LOGIC_SIGNAL: track 8.74 -> 0.00 mm
- net /A9G_GSM_GPRS_MODULE/GPS_RXD: track 66.2 -> 57.5 mm
- net /A9G_GSM_GPRS_MODULE/IO29: track 47.2 -> 55.6 mm
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
Commit message: all items updated
Parts:
- removed AE3: Antenna_Shield, greencharge-footprints:UFL_COAX_CONN23370191
- removed J4: Micro_SD_Card, MACHADA_footprints:MOLEX_503398-1892
- removed R47: 10k, Resistor_SMD:R_0402_1005Metric
- removed U10, U12, U18, U20, U4, U6: TBU-CA065-200-WH, MACHADA_footprints:TBU-CA065-200-WH
- added C37: 0.1u, Capacitor_SMD:C_0402_1005Metric, F.Cu at (93.0, 90.0)
- added C38: 1u, Capacitor_SMD:C_0402_1005Metric, F.Cu at (91.9, 90.0)
- added D19: 4.4-4.5 ZENER, Diode_SMD:D_SOD-123, B.Cu at (60.2, 84.4)
- added J7: Micro_SD_Card, MACHADA_footprints:MOLEX_503398-1892, B.Cu at (87.2, 91.5)
- added L3: ferrite bead, Inductor_SMD:L_0402_1005Metric, F.Cu at (52.4, 91.0)
- added L4: ferrite bead, Inductor_SMD:L_0402_1005Metric, F.Cu at (52.3, 101.2)
- added L6: ferrite bead, Inductor_SMD:L_0402_1005Metric, F.Cu at (43.1, 117.0)
- added L7: ferrite bead, Inductor_SMD:L_0402_1005Metric, F.Cu at (52.1, 89.2)
- added L8: ferrite bead, Inductor_SMD:L_0402_1005Metric, F.Cu at (52.4, 99.8)
- added L9: ferrite bead, Inductor_SMD:L_0402_1005Metric, F.Cu at (41.5, 117.0)
- added R17: 22R, Resistor_SMD:R_0402_1005Metric, F.Cu at (70.4, 62.4)
- added R18: 49.9R, Resistor_SMD:R_0402_1005Metric, B.Cu at (62.4, 86.2)
- added R19: 10k, Resistor_SMD:R_0402_1005Metric, F.Cu at (55.4, 86.1)
- AE1: footprint Connector_Coaxial:SMA_Samtec_SMA-J-P-X-ST-EM1_EdgeMount -> Connector_Coaxial:SMA_Molex_73251-2200_Horizontal
- C21: value 0.1u -> C_Small; moved to F.Cu
- C22: value 1u -> C_Small; moved to F.Cu
- C46, C58: footprint Capacitor_SMD:C_0603_1608Metric -> Capacitor_SMD:C_0402_1005Metric
- D10: value SS310 -> RS1K-E3/5ATSS310
- D2: footprint LED_SMD:LED_0603_1608Metric -> LED_SMD:LED_0402_1005Metric
- H4: moved to B.Cu
- L1: footprint Inductor_SMD:L_0603_1608Metric -> Inductor_SMD:L_0402_1005Metric
- Q5, Q6: value BSN20 -> IRLML0100TRPBF
- TH1: footprint Fuse:Fuse_0603_1608Metric_Pad1.05x0.95mm_HandSolder -> Fuse:Fuse_1206_3216Metric
- moved R8 45.2 mm to (65.8, 59.6), turned to -90 degrees
- moved D2 44.9 mm to (64.8, 59.6), turned to -90 degrees
- moved C22 39.7 mm to (43.5, 70.7), turned to 90 degrees
- moved C21 35.9 mm to (46.8, 70.7), turned to 90 degrees
- moved D+1 29.9 mm to (40.6, 62.6)
- moved HST_TXD1 22.3 mm to (40.2, 60.1)
- moved C15 21.4 mm to (76.5, 69.6)
- moved C16 21.4 mm to (72.8, 73.6)
- moved C17 21.4 mm to (71.7, 73.6)
- moved C14 21.4 mm to (76.5, 70.7)
- moved U17 21.4 mm to (75.4, 73.0)
- moved D5 19.1 mm to (59.4, 59.6)
- moved R35 18.8 mm to (58.2, 59.6)
- moved R34 17.5 mm to (72.2, 82.4), turned to 180 degrees
- moved AE1 17.3 mm to (75.1, 61.9), turned to -90 degrees
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Connections:
- C21 pad 1: 2V8 -> GND
- C21 pad 2: GND -> Net-(U3-GSM_RF)
- C22 pad 1: 2V8 -> GND
- C22 pad 2: GND -> Net-(AE2-A)
- L2 pad 1: Net-(AE1-A) -> Net-(L2-Pad1)
- R40 pad 2: /A9G_GSM_GPRS_MODULE/TF_CARD_CONN/SD_D2 -> /A9G_GSM_GPRS_MODULE/TF_CARD_CONN/SD_D3
- R41 pad 2: /A9G_GSM_GPRS_MODULE/TF_CARD_CONN/SD_D3 -> /A9G_GSM_GPRS_MODULE/TF_CARD_CONN/SD_CMD
- R42 pad 2: /A9G_GSM_GPRS_MODULE/TF_CARD_CONN/SD_CMD -> /A9G_GSM_GPRS_MODULE/TF_CARD_CONN/SD_D0
- R45 pad 2: /A9G_GSM_GPRS_MODULE/TF_CARD_CONN/SD_D0 -> /A9G_GSM_GPRS_MODULE/TF_CARD_CONN/SD_D1
- R46 pad 2: /A9G_GSM_GPRS_MODULE/TF_CARD_CONN/SD_D1 -> /A9G_GSM_GPRS_MODULE/TF_CARD_CONN/SD_CLK
- U1 pad 12: /A9G_GSM_GPRS_MODULE/GPS_TXD -> /A9G_GSM_GPRS_MODULE/GPS_RXD
- U1 pad 13: /A9G_GSM_GPRS_MODULE/GPS_RXD -> /A9G_GSM_GPRS_MODULE/GPS_TXD
- U1 pad 21: /STM32FC8T6_MCU/RS485_RO -> /MULTIPLEXER_SWITCH_WAS3157B-6/SIG1_IN
- U1 pad 22: /STM32FC8T6_MCU/RS485_DI -> /MULTIPLEXER_SWITCH_WAS3157B-6/SIG2_IN
- U1 pad 32: /MULTIPLEXER_SWITCH_WAS3157B-6/SIG2_IN -> /STM32FC8T6_MCU/RS485_DI
- U1 pad 33: /MULTIPLEXER_SWITCH_WAS3157B-6/SIG1_IN -> /STM32FC8T6_MCU/RS485_RO
- U3 pad 49: /A9G_GSM_GPRS_MODULE/GPS_RXD -> /A9G_GSM_GPRS_MODULE/GPS_TXD
- U3 pad 50: /A9G_GSM_GPRS_MODULE/GPS_TXD -> /A9G_GSM_GPRS_MODULE/GPS_RXD
- U3 pad 53: /STM32FC8T6_MCU/RX1 -> /STM32FC8T6_MCU/TX1
- U3 pad 54: /STM32FC8T6_MCU/TX1 -> /STM32FC8T6_MCU/RX1
Routing:
- net /STM32FC8T6_MCU/3v3_stm: track 113.6 -> 191.5 mm, vias 9 -> 14
- net Net-(D2-K): track 39.9 -> 113.4 mm, vias 2 -> 4
- net /A9G_GSM_GPRS_MODULE/Sim_Restart: track 67.7 -> 46.6 mm, vias 2 -> 4
- net /MULTIPLEXER_SWITCH_WAS3157B-6/SIG2_IN: track 27.8 -> 48.6 mm, vias 2 -> 3
- net /A9G_GSM_GPRS_MODULE/V_Sim: track 22.5 -> 41.5 mm
- net Net-(U3-USB_P): track 3.58 -> 22.2 mm, vias 0 -> 2
- net /A9G_GSM_GPRS_MODULE/GPS_RXD: track 57.5 -> 75.3 mm
- net /A9G_GSM_GPRS_MODULE/PWRKEY: track 28.4 -> 45.6 mm
- net /A9G_GSM_GPRS_MODULE/IO29: track 55.6 -> 38.8 mm
- net Net-(J2-RST): track 34.4 -> 51.0 mm
- net 4.2V_SIMPWR: track 46.7 -> 30.7 mm, vias 9 -> 8
- net /A9G_GSM_GPRS_MODULE/TF_CARD_CONN/SD_D0: track 28.7 -> 44.3 mm
- net Net-(J2-CLK): track 26.6 -> 41.7 mm
- net Net-(U3-HST_RXD): track 10.9 -> 26.0 mm, vias 0 -> 2
- net 2V8: track 62.8 -> 77.8 mm, vias 3 -> 5
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- added copper zone on B.Cu, net +5V
Other:
- outline, holes or cut-outs redrawn
