File: SOURCE_FILES/BIM_PCB/BIM_PCB.kicad_pcb (KiCad board)
At the start: 4 copper layers, 58.5 x 72.5 mm, 199 parts, among them J1 Conn_02x09_Counter_Clockwise, J2 nano_sim, J3 Conn_01x06, J7 Micro_SD_Card, Q1 SSM3J328R-HXY, Q2 SSM3J328R-HXY, Q3 IRLML0100TRPBF, Q5 IRLML0100TRPBF, Q6 IRLML0100TRPBF, SW1 reset, U1 STM32F103C8Tx, U11 SSP3485U, U13 ATA6561-GAQW-N, U14 WAS3157B, U15 MC74HC4052A, U16 SY8089AAAC, U17 XC6206PxxxMR, U19 SSP3485U, U2 PCF8523TK, U3 A9G_MODULE, U5 SSP3485U, U7 WAS3157B, U8 W25Q32JVSS, U9 ATA6561-GAQW-N, Y1 8MHz, Y2 32.678KHz, Y3 32.678KHz

Commit message: all items updated
Parts:
- U14, U7: value WAS3157B -> SN74LVC1G3157DBVR
- moved R36 2.82 mm to (58.4, 59.6)
- moved R35 1.96 mm to (60.2, 59.6)
- moved D5 1.91 mm to (61.4, 59.6)
- moved D2 0.83 mm to (64.0, 59.6), turned to 90 degrees
- moved R8 0.54 mm to (65.3, 59.6), turned to 90 degrees
Connections:
- U1 pad 21: /MULTIPLEXER_SWITCH_WAS3157B-6/SIG1_IN -> /STM32FC8T6_MCU/RS485_DI
- U1 pad 22: /MULTIPLEXER_SWITCH_WAS3157B-6/SIG2_IN -> /STM32FC8T6_MCU/RS485_RO
- U1 pad 32: /STM32FC8T6_MCU/RS485_DI -> /MULTIPLEXER_SWITCH_WAS3157B-6/SIG2_IN
- U1 pad 33: /STM32FC8T6_MCU/RS485_RO -> /MULTIPLEXER_SWITCH_WAS3157B-6/SIG1_IN
Routing:
- net /MULTIPLEXER_SWITCH_WAS3157B-6/SIG2_IN: track 48.6 -> 40.3 mm
- net /RS485_B: track 9.14 -> 15.4 mm
- net /MULTIPLEXER_SWITCH_WAS3157B-6/SIG1_IN: track 26.5 -> 21.5 mm
- net Net-(D6-A): track 1.30 -> 5.55 mm
- net Net-(D18-K-Pad2): track 16.1 -> 19.4 mm
- net /STM32FC8T6_MCU/RS485_RO: track 48.7 -> 51.1 mm
- net GND: track 156.0 -> 158.3 mm, vias 661 -> 660
- net /A9G_GSM_GPRS_MODULE/GPS POSITION: track 7.46 -> 9.63 mm
- net /DIS_A: track 34.8 -> 36.6 mm
- net Net-(D15-K-Pad2): track 17.3 -> 19.1 mm
- net /A9G_GSM_GPRS_MODULE/GPRS_NET-STATUS: track 20.6 -> 22.2 mm
- net /STM32FC8T6_MCU/3v3_stm: track 191.5 -> 192.8 mm
- net /STM32FC8T6_MCU/RS485_DI: track 34.4 -> 35.6 mm
- net Net-(D15-K-Pad1): track 18.3 -> 19.2 mm
- net /SCL: track 26.9 -> 26.2 mm
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
Commit message: all items updated including fiducial
Parts:
- added REF**: Fiducial_1.5mm_Mask3mm, Fiducial:Fiducial_1.5mm_Mask3mm, F.Cu at (86.2, 123.7)
- added REF**: Fiducial_1.5mm_Mask3mm, Fiducial:Fiducial_1.5mm_Mask3mm, F.Cu at (40.9, 121.2)
- added REF**: Fiducial_1.5mm_Mask3mm, Fiducial:Fiducial_1.5mm_Mask3mm, F.Cu at (91.0, 70.5)
- added REF**: Fiducial_1.5mm_Mask3mm, Fiducial:Fiducial_1.5mm_Mask3mm, B.Cu at (75.1, 66.7)
- added REF**: Fiducial_1.5mm_Mask3mm, Fiducial:Fiducial_1.5mm_Mask3mm, B.Cu at (43.1, 121.0)
- added REF**: Fiducial_1.5mm_Mask3mm, Fiducial:Fiducial_1.5mm_Mask3mm, B.Cu at (82.4, 125.2)
