File: SOURCE_FILES/BIM_PCB/TF_CARD_CONN.kicad_sch (KiCad schematic)
At the start: 9 parts, among them J7 Micro_SD_Card

Commit message: updated GENERAL
Other:
- note added: "TF/SD CARD"
Changed lines of the file:
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@@
     (stroke (width 0) (type default))
+  )
+  (text "TF/SD CARD" (at 120.65 36.83 0)
+    (effects (font (face "Agency FB") (size 6 6) (thickness 1.2) bold) (justify left bottom))
   )
   (label "2V8" (at 152.4 86.36 0) (fields_autoplaced)

Commit message: completed project
Changed lines of the file:
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@@
-    (effects (font (size 1.27 1.27)) (justify left bottom))
-  )
-  (label "2V8" (at 157.48 60.96 0) (fields_autoplaced)
     (effects (font (size 1.27 1.27)) (justify left bottom))
   )
@@
     (effects (font (size 1.27 1.27)) (justify right))
   )
+  (hierarchical_label "2V8" (shape input) (at 157.48 60.96 0) (fields_autoplaced)
+    (effects (font (size 1.27 1.27)) (justify left))
+  )
   (hierarchical_label "SD_D2" (shape bidirectional) (at 137.795 85.09 0) (fields_autoplaced)

Commit message: all items updated
Parts:
- removed C44: 1u, Capacitor_SMD:C_0402_1005Metric, symbol fridgeduino-rescue:C_Small-Device
- removed C45: 0.1u, Capacitor_SMD:C_0402_1005Metric, symbol fridgeduino-rescue:C_Small-Device
- removed R44 (x3), R47: 10k, Resistor_SMD:R_0402_1005Metric, symbol fridgeduino-rescue:R_Small_US-Device
- added C37: 0.1u, Capacitor_SMD:C_0402_1005Metric, symbol fridgeduino-rescue:C_Small-Device
- added C38: 1u, Capacitor_SMD:C_0402_1005Metric, symbol fridgeduino-rescue:C_Small-Device
- added R19, R40, R41, R42: 10k, Resistor_SMD:R_0402_1005Metric, symbol fridgeduino-rescue:R_Small_US-Device
Connections:
- net 2V8: now also C37.1, C38.1, R19.1, R40.1, R41.1, R42.1
- net GND: now also C37.2, C38.2
- net SD_CLK: now also R46.2
- net SD_CMD: now also R41.2; no longer R45.2
- net SD_D0: now also R42.2
- net SD_D1: now also R45.2
- net SD_D2: now also R19.2
- net SD_D3: now also R40.2; no longer R46.2
