File: SOURCE_FILES/BIM_PCB/BIM_PCB.kicad_sch (KiCad schematic)
At the start: 18 parts, among them J1 Conn_02x09_Counter_Clockwise, Q1 SSM3J328R-HXY, Q2 SSM3J328R-HXY, Q6 IRLML0100TRPBF, U15 MC74HC4052A

Commit message: completed BIM board- ECOBoda
Parts:
- added J5: Conn_02x06_Odd_Even, MACHADA_footprints:auto_jae_conn_02x06_p2.5mm_MX23A12NF1, symbol Connector_Generic:Conn_02x06_Odd_Even
- J1: footprint MACHADA_footprints:conn_18pin_02x09_angled_MX23A18NF1 -> MACHADA_footprints:auto_jae_conn_02x06_p2.5mm_MX23A12NF1; MPN MX23A18NF1 -> MX23A12NF1
Changed lines of the file:
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@@
       (effects (font (size 1.27 1.27)))
     )
-    (property "Footprint" "MACHADA_footprints:conn_18pin_02x09_angled_MX23A18NF1" (at 375.92 229.87 0)
+    (property "Footprint" "MACHADA_footprints:auto_jae_conn_02x06_p2.5mm_MX23A12NF1" (at 375.92 229.87 0)
       (effects (font (size 1.27 1.27)) hide)
     )
@@
       (effects (font (size 1.27 1.27)) hide)
     )
-    (property "MPN" "MX23A18NF1" (at 391.16 216.535 0)
+    (property "MPN" "MX23A12NF1" (at 391.16 216.535 0)
       (effects (font (size 1.27 1.27)))
     )
@@
         )
       )
+    )
+  )
+  (symbol (lib_id "Connector_Generic:Conn_02x06_Odd_Even") (at 398.145 156.21 0) (unit 1)
+    (in_bom yes) (on_board yes) (dnp no)
+    (property "Reference" "J5" (at 399.415 144.78 0)
+      (effects (font (size 1.27 1.27)))
+    )
+    (property "Value" "Conn_02x06_Odd_Even" (at 399.415 147.32 0)
+      (effects (font (size 1.27 1.27)))
+    )
+    (property "Footprint" "MACHADA_footprints:auto_jae_conn_02x06_p2.5mm_MX23A12NF1" (at 398.145 156.21 0)
+      (effects (font (size 1.27 1.27)) hide)
+    )
+    (property "Datasheet" "~" (at 398.145 156.21 0)
+      (effects (font (size 1.27 1.27)) hide)
+    )
+    (property "MPN" "MX23A12NF1" (at 399.415 167.005 0)
+      (effects (font (size 1.27 1.27)))
+    )
+    (pin "8")
+    (pin "5")
+    (pin "1")
+    (pin "3")
+    (pin "2")
+    (pin "6")
+    (pin "7")
+    (pin "4")
+    (pin "9")
+    (pin "12")
+    (pin "11")
+    (pin "10")
+    (instances
+      (project "BIM_PCB"
+        (path "/b79ebed7-e146-448b-8dab-0aefb3e182ca"
+          (reference "J5") (unit 1)
+        )
+      )

Commit message: completed project and all the prouction files
Parts:
- removed J5: Conn_02x06_Odd_Even, MACHADA_footprints:auto_jae_conn_02x06_p2.5mm_MX23A12NF1, symbol Connector_Generic:Conn_02x06_Odd_Even
- C46: footprint Capacitor_SMD:C_0603_1608Metric -> Capacitor_SMD:C_0402_1005Metric
- D10: value SS310 -> RS1K-E3/5ATSS310
- J1: footprint MACHADA_footprints:auto_jae_conn_02x06_p2.5mm_MX23A12NF1 -> MACHADA_footprints:conn_18pin_02x09_angled_MX23A18NF1; MPN MX23A12NF1 -> MX23A18NF1
Changed lines of the file:
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@@
       (effects (font (size 1.27 1.27)))
     )
-    (property "Footprint" "MACHADA_footprints:auto_jae_conn_02x06_p2.5mm_MX23A12NF1" (at 375.92 229.87 0)
+    (property "Footprint" "MACHADA_footprints:conn_18pin_02x09_angled_MX23A18NF1" (at 375.92 229.87 0)
       (effects (font (size 1.27 1.27)) hide)
     )
@@
       (effects (font (size 1.27 1.27)) hide)
     )
-    (property "MPN" "MX23A12NF1" (at 391.16 216.535 0)
+    (property "MPN" "MX23A18NF1" (at 391.16 216.535 0)
       (effects (font (size 1.27 1.27)))
     )
@@
   (symbol (lib_id "Device:Q_NMOS_GSD") (at 250.825 231.14 0) (unit 1)
     (in_bom yes) (on_board yes) (dnp no) (fields_autoplaced)
-    (property "Reference" "Q6" (at 257.175 230.505 0)
-      (effects (font (size 1.27 1.27)) (justify left))
-    )
-    (property "Value" "IRLML0100TRPBF" (at 257.175 233.045 0)
+    (property "Reference" "Q6" (at 256.54 229.87 0)
+      (effects (font (size 1.27 1.27)) (justify left))
+    )
+    (property "Value" "IRLML0100TRPBF" (at 256.54 232.41 0)
       (effects (font (size 1.27 1.27)) (justify left))
     )
@@
     )
   )
-  (symbol (lib_id "Connector_Generic:Conn_02x06_Odd_Even") (at 398.145 156.21 0) (unit 1)
-    (in_bom yes) (on_board yes) (dnp no)
-    (property "Reference" "J5" (at 399.415 144.78 0)
-      (effects (font (size 1.27 1.27)))
-    )
-    (property "Value" "Conn_02x06_Odd_Even" (at 399.415 147.32 0)
-      (effects (font (size 1.27 1.27)))
-    )
-    (property "Footprint" "MACHADA_footprints:auto_jae_conn_02x06_p2.5mm_MX23A12NF1" (at 398.145 156.21 0)
-      (effects (font (size 1.27 1.27)) hide)
-    )
-    (property "Datasheet" "~" (at 398.145 156.21 0)
-      (effects (font (size 1.27 1.27)) hide)
-    )
-    (property "MPN" "MX23A12NF1" (at 399.415 167.005 0)
-      (effects (font (size 1.27 1.27)))
-    )
-    (pin "8")
-    (pin "5")
-    (pin "1")
-    (pin "3")
-    (pin "2")
-    (pin "6")
-    (pin "7")
-    (pin "4")
-    (pin "9")
-    (pin "12")
-    (pin "11")
-    (pin "10")
-    (instances
-      (project "BIM_PCB"
-        (path "/b79ebed7-e146-448b-8dab-0aefb3e182ca"
-          (reference "J5") (unit 1)
-        )
-      )
-    )
-  )
   (symbol (lib_id "power:GND") (at 245.745 123.19 0) (mirror y) (unit 1)
     (in_bom yes) (on_board yes) (dnp no)
@@
       (effects (font (size 1.27 1.27)) (justify left))
     )
-    (property "Footprint" "Capacitor_SMD:C_0603_1608Metric" (at 245.745 120.65 0)
+    (property "Footprint" "Capacitor_SMD:C_0402_1005Metric" (at 245.745 120.65 0)
       (effects (font (size 1.27 1.27)) hide)
     )
@@
   (symbol (lib_id "Device:D_Schottky") (at 219.71 26.67 180) (unit 1)
     (in_bom yes) (on_board yes) (dnp no) (fields_autoplaced)
-    (property "Reference" "D10" (at 220.0275 20.955 0)
-      (effects (font (size 1.27 1.27)))
-    )
-    (property "Value" "SS310" (at 220.0275 23.495 0)
-      (effects (font (size 1.27 1.27)))
-    )
+    (property "Reference" "D10" (at 220.0275 20.32 0)
+      (effects (font (size 1.27 1.27)))
+    )
+    (property "Value" "RS1K-E3/5ATSS310" (at 220.0275 22.86 0)
+      (effects (font (size 1.27 1.27)))
+    )

Commit message: all items updated
Parts:
- added D19: 4.4-4.5 ZENER, Diode_SMD:D_SOD-123, symbol Diode:BZV55C10
- added R18: 49.9R, Resistor_SMD:R_0402_1005Metric, symbol Device:R_US
- TH1: footprint Fuse:Fuse_0603_1608Metric_Pad1.05x0.95mm_HandSolder -> Fuse:Fuse_1206_3216Metric; MPN PRG18BC1R0MM1RB -> ASMD1206-100
Connections:
- net 4.2V_SIMPWR: now also D19.1 (K)
- net GND: now also R18.2
- new net: D19.2 (A), R18.1
Other:
- sheet STM32FC8T6_MCU ports: added RX1, RXD, TX1, TXD; removed GPS_RXD, GPS_TXD, Sim_Rx, Sim_Tx
- moved on the sheet: SIM_PWR1
Changed lines of the file:
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@@
   (junction (at 73.66 34.925) (diameter 0) (color 0 0 0 0)
+  )
+  (junction (at 257.175 27.94) (diameter 0) (color 0 0 0 0)
   )
   (junction (at 118.11 34.925) (diameter 0) (color 0 0 0 0)
@@
     (stroke (width 0) (type default))
   )
+  (wire (pts (xy 257.175 26.67) (xy 257.048 26.67))
+    (stroke (width 0) (type default))
+  )
   (wire (pts (xy 66.04 91.44) (xy 127 91.44))
     (stroke (width 0) (type default))
@@
     (stroke (width 0) (type default))
   )
-  (wire (pts (xy 257.048 27.178) (xy 257.048 26.67))
+  (wire (pts (xy 257.175 27.94) (xy 257.175 26.67))
     (stroke (width 0) (type default))
   )
@@
     (stroke (width 0) (type default))
   )
+  (wire (pts (xy 257.175 43.18) (xy 257.175 45.72))
+    (stroke (width 0) (type default))
+  )
   (wire (pts (xy 301.625 127) (xy 311.15 127))
     (stroke (width 0) (type default))
@@
     (stroke (width 0) (type default))
   )
+  (wire (pts (xy 257.175 27.94) (xy 260.985 27.94))
+    (stroke (width 0) (type default))
+  )
   (wire (pts (xy 162.56 158.115) (xy 170.815 158.115))
     (stroke (width 0) (type default))
@@
   )
   (wire (pts (xy 264.795 145.415) (xy 246.38 145.415))
-    (stroke (width 0) (type default))
-  )
-  (wire (pts (xy 260.858 27.178) (xy 257.048 27.178))
     (stroke (width 0) (type default))
   )
@@
       (effects (font (size 1.27 1.27)))
     )
-    (property "Footprint" "Fuse:Fuse_0603_1608Metric_Pad1.05x0.95mm_HandSolder" (at 55.88 33.655 0)
+    (property "Footprint" "Fuse:Fuse_1206_3216Metric" (at 55.88 33.655 0)
       (effects (font (size 1.27 1.27)) (justify left) hide)
     )
@@
       (effects (font (size 1.27 1.27)) hide)
     )
-    (property "MPN" "PRG18BC1R0MM1RB" (at 50.8 38.735 90)
+    (property "MPN" "ASMD1206-100" (at 50.8 38.735 90)
       (effects (font (size 1.27 1.27)))
     )
@@
         (path "/b79ebed7-e146-448b-8dab-0aefb3e182ca"
           (reference "#PWR082") (unit 1)
+        )
+      )
+    )
+  )
+  (symbol (lib_id "Diode:BZV55C10") (at 257.175 31.75 270) (unit 1)
+    (in_bom yes) (on_board yes) (dnp no) (fields_autoplaced)
+    (property "Reference" "D19" (at 260.35 30.48 90)
+      (effects (font (size 1.27 1.27)) (justify left))
+    )
+    (property "Value" "4.4-4.5 ZENER" (at 260.35 33.02 90)
+      (effects (font (size 1.27 1.27)) (justify left))
+    )
+    (property "Footprint" "Diode_SMD:D_SOD-123" (at 252.73 31.75 0)
+      (effects (font (size 1.27 1.27)) hide)
+    )
+    (property "Datasheet" "https://assets.nexperia.com/documents/data-sheet/BZV55_SER.pdf" (at 257.175 31.75 0)
+      (effects (font (size 1.27 1.27)) hide)
+    )
+    (pin "1")
+    (pin "2")
+    (instances
+      (project "BIM_PCB"
+        (path "/b79ebed7-e146-448b-8dab-0aefb3e182ca"
+          (reference "D19") (unit 1)
         )
       )
@@
     )
   )
-  (symbol (lib_id "Connector:TestPoint") (at 260.858 27.178 0) (mirror y) (unit 1)
+  (symbol (lib_id "Connector:TestPoint") (at 260.985 27.94 0) (mirror y) (unit 1)
     (in_bom yes) (on_board yes) (dnp no)
-    (property "Reference" "SIM_PWR1" (at 267.716 24.638 0)
-      (effects (font (size 1.27 1.27)))
-    )
-    (property "Value" "TestPoint" (at 267.081 22.733 0)
-      (effects (font (size 1.27 1.27)))
-    )
-    (property "Footprint" "brilliant-kicad-library:TestPoint_Pad_D0.9mm" (at 255.778 27.178 0)
-      (effects (font (size 1.27 1.27)) hide)
-    )
-    (property "Datasheet" "~" (at 255.778 27.178 0)
+    (property "Reference" "SIM_PWR1" (at 267.843 25.4 0)
+      (effects (font (size 1.27 1.27)))
+    )
+    (property "Value" "TestPoint" (at 267.208 23.495 0)
+      (effects (font (size 1.27 1.27)))
+    )
+    (property "Footprint" "brilliant-kicad-library:TestPoint_Pad_D0.9mm" (at 255.905 27.94 0)
+      (effects (font (size 1.27 1.27)) hide)
+    )
+    (property "Datasheet" "~" (at 255.905 27.94 0)
       (effects (font (size 1.27 1.27)) hide)
     )
@@
     )
   )
+  (symbol (lib_id "power:GND") (at 257.175 45.72 0) (unit 1)
+    (in_bom yes) (on_board yes) (dnp no) (fields_autoplaced)
+    (property "Reference" "#PWR031" (at 257.175 52.07 0)
+      (effects (font (size 1.27 1.27)) hide)
+    )
+    (property "Value" "GND" (at 257.175 50.8 0)
+      (effects (font (size 1.27 1.27)))
+    )
+    (property "Footprint" "" (at 257.175 45.72 0)
+      (effects (font (size 1.27 1.27)) hide)
+    )
+    (property "Datasheet" "" (at 257.175 45.72 0)
+      (effects (font (size 1.27 1.27)) hide)
+    )
+    (pin "1")
+    (instances
+      (project "BIM_PCB"
+        (path "/b79ebed7-e146-448b-8dab-0aefb3e182ca"
+          (reference "#PWR031") (unit 1)
+        )
+      )
+    )
+  )
   (symbol (lib_id "Device:D_Schottky") (at 219.71 26.67 180) (unit 1)
     (in_bom yes) (on_board yes) (dnp no) (fields_autoplaced)
@@
         (path "/f580900f-d859-42c8-b556-7826c8dbedd6"
           (reference "D12") (unit 1)
+        )
+      )
+    )
+  )
+  (symbol (lib_id "Device:R_US") (at 257.175 39.37 0) (unit 1)
+    (in_bom yes) (on_board yes) (dnp no) (fields_autoplaced)
+    (property "Reference" "R18" (at 259.715 38.735 0)
+      (effects (font (size 1.27 1.27)) (justify left))
+    )
+    (property "Value" "49.9R" (at 259.715 41.275 0)
+      (effects (font (size 1.27 1.27)) (justify left))
+    )
+    (property "Footprint" "Resistor_SMD:R_0402_1005Metric" (at 258.191 39.624 90)
+      (effects (font (size 1.27 1.27)) hide)
+    )
+    (property "Datasheet" "~" (at 257.175 39.37 0)
+      (effects (font (size 1.27 1.27)) hide)
+    )
+    (pin "1")
+    (pin "2")
+    (instances
+      (project "BIM_PCB"
+        (path "/b79ebed7-e146-448b-8dab-0aefb3e182ca"
+          (reference "R18") (unit 1)
         )
       )
@@
       (effects (font (size 1.27 1.27)) (justify right))
     )
+    (pin "Sim_Rx" input (at 66.04 99.06 0)
+      (effects (font (size 1.27 1.27)) (justify right))
+    )
+    (pin "Sim_Tx" output (at 66.04 101.6 0)
+      (effects (font (size 1.27 1.27)) (justify right))
+    )
+    (pin "GPS_RXD" input (at 66.04 111.125 0)
+      (effects (font (size 1.27 1.27)) (justify right))
+    )
     (pin "GPS_TXD" output (at 66.04 114.3 0)
-      (effects (font (size 1.27 1.27)) (justify right))
-    )
-    (pin "GPS_RXD" input (at 66.04 111.125 0)
-      (effects (font (size 1.27 1.27)) (justify right))
-    )
-    (pin "Sim_Rx" input (at 66.04 99.06 0)
-      (effects (font (size 1.27 1.27)) (justify right))
-    )
-    (pin "Sim_Tx" output (at 66.04 101.6 0)
       (effects (font (size 1.27 1.27)) (justify right))
     )
@@
       (effects (font (size 1.27 1.27)) (justify right))
     )
-    (pin "Sim_Tx" output (at 127 99.06 180)
-      (effects (font (size 1.27 1.27)) (justify left))
-    )
-    (pin "Sim_Rx" input (at 127 101.6 180)
-      (effects (font (size 1.27 1.27)) (justify left))
-    )
     (pin "SCK" output (at 127 156.21 180)
       (effects (font (size 1.27 1.27)) (justify left))
@@
       (effects (font (size 1.27 1.27)) (justify right))
     )
-    (pin "GPS_TXD" output (at 127 111.125 180)
-      (effects (font (size 1.27 1.27)) (justify left))
-    )
-    (pin "GPS_RXD" input (at 127 114.3 180)
-      (effects (font (size 1.27 1.27)) (justify left))
-    )
     (pin "RS485_~{RE}" output (at 162.56 155.575 0)
       (effects (font (size 1.27 1.27)) (justify right))
@@
       (effects (font (size 1.27 1.27)) (justify right))
     )
-    (instances
+    (pin "RXD" input (at 127 114.3 180)
+      (effects (font (size 1.27 1.27)) (justify left))
+    )
+    (pin "TXD" output (at 127 111.125 180)
+      (effects (font (size 1.27 1.27)) (justify left))
+    )
+    (pin "TX1" output (at 127 99.06 180)
+      (effects (font (size 1.27 1.27)) (justify left))
+    )
+    (pin "RX1" input (at 127 101.6 180)
+      (effects (font (size 1.27 1.27)) (justify left))
+    )
+    (instances
