File: SOURCE_FILES/BIM_PCB/BIM_PCB.kicad_sch (KiCad schematic)
At the start: 20 parts, among them J1 Conn_02x09_Counter_Clockwise, Q1 SSM3J328R-HXY, Q2 SSM3J328R-HXY, Q6 IRLML0100TRPBF, U15 MC74HC4052A

Commit message: all items updated
Parts:
- D11, D12: value SS310 -> RS1K-E3/5ATSS310
Other:
- moved on the sheet: D11, D12, D19, R18, SIM_PWR1
Changed lines of the file:
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@@
   (junction (at 73.66 34.925) (diameter 0) (color 0 0 0 0)
   )
-  (junction (at 257.175 27.94) (diameter 0) (color 0 0 0 0)
+  (junction (at 281.94 27.94) (diameter 0) (color 0 0 0 0)
   )
   (junction (at 118.11 34.925) (diameter 0) (color 0 0 0 0)
@@
   (junction (at 77.47 34.925) (diameter 0) (color 0 0 0 0)
   )
-  (junction (at 257.048 26.67) (diameter 0) (color 0 0 0 0)
+  (junction (at 281.813 26.67) (diameter 0) (color 0 0 0 0)
   )
   (junction (at 77.47 48.895) (diameter 0) (color 0 0 0 0)
@@
     (stroke (width 0) (type default))
   )
-  (wire (pts (xy 257.175 26.67) (xy 257.048 26.67))
+  (wire (pts (xy 281.94 26.67) (xy 281.813 26.67))
     (stroke (width 0) (type default))
   )
@@
     (stroke (width 0) (type default))
   )
-  (wire (pts (xy 257.175 27.94) (xy 257.175 26.67))
+  (wire (pts (xy 281.94 27.94) (xy 281.94 26.67))
     (stroke (width 0) (type default))
   )
@@
     (stroke (width 0) (type default))
   )
-  (wire (pts (xy 257.175 43.18) (xy 257.175 45.72))
+  (wire (pts (xy 281.94 43.18) (xy 281.94 45.72))
     (stroke (width 0) (type default))
   )
@@
     (stroke (width 0) (type default))
   )
-  (wire (pts (xy 247.015 26.67) (xy 237.49 26.67))
+  (wire (pts (xy 265.43 26.67) (xy 250.19 26.67))
     (stroke (width 0) (type default))
   )
@@
     (stroke (width 0) (type default))
   )
-  (wire (pts (xy 257.175 27.94) (xy 260.985 27.94))
+  (wire (pts (xy 281.94 27.94) (xy 285.75 27.94))
     (stroke (width 0) (type default))
   )
@@
     (stroke (width 0) (type default))
   )
-  (wire (pts (xy 254.635 26.67) (xy 257.048 26.67))
+  (wire (pts (xy 273.05 26.67) (xy 281.813 26.67))
     (stroke (width 0) (type default))
   )
@@
     (stroke (width 0) (type default))
   )
-  (wire (pts (xy 229.87 26.67) (xy 223.52 26.67))
+  (wire (pts (xy 242.57 26.67) (xy 223.52 26.67))
     (stroke (width 0) (type default))
   )
@@
     (stroke (width 0) (type default))
   )
-  (wire (pts (xy 257.048 18.288) (xy 257.048 26.67))
+  (wire (pts (xy 281.813 18.288) (xy 281.813 26.67))
     (stroke (width 0) (type default))
   )
@@
     )
   )
-  (global_label "4.2V_SIMPWR" (shape input) (at 257.048 18.288 0) (fields_autoplaced)
+  (global_label "4.2V_SIMPWR" (shape input) (at 281.813 18.288 0) (fields_autoplaced)
     (effects (font (size 1.27 1.27)) (justify left))
-    (property "Intersheetrefs" "${INTERSHEET_REFS}" (at 272.2909 18.288 0)
+    (property "Intersheetrefs" "${INTERSHEET_REFS}" (at 297.0559 18.288 0)
       (effects (font (size 1.27 1.27)) (justify left) hide)
     )
@@
     )
   )
-  (symbol (lib_id "Device:D_Schottky") (at 233.68 26.67 180) (unit 1)
-    (in_bom yes) (on_board yes) (dnp no) (fields_autoplaced)
-    (property "Reference" "D11" (at 233.9975 20.955 0)
-      (effects (font (size 1.27 1.27)))
-    )
-    (property "Value" "SS310" (at 233.9975 23.495 0)
-      (effects (font (size 1.27 1.27)))
-    )
-    (property "Footprint" "Diode_SMD:D_SMA" (at 233.68 26.67 0)
-      (effects (font (size 1.27 1.27)) hide)
-    )
-    (property "Datasheet" "~" (at 233.68 26.67 0)
+  (symbol (lib_id "Device:D_Schottky") (at 246.38 26.67 180) (unit 1)
+    (in_bom yes) (on_board yes) (dnp no) (fields_autoplaced)
+    (property "Reference" "D11" (at 246.6975 20.32 0)
+      (effects (font (size 1.27 1.27)))
+    )
+    (property "Value" "RS1K-E3/5ATSS310" (at 246.6975 22.86 0)
+      (effects (font (size 1.27 1.27)))
+    )
+    (property "Footprint" "Diode_SMD:D_SMA" (at 246.38 26.67 0)
+      (effects (font (size 1.27 1.27)) hide)
+    )
+    (property "Datasheet" "~" (at 246.38 26.67 0)
       (effects (font (size 1.27 1.27)) hide)
     )
@@
     )
   )
-  (symbol (lib_id "Diode:BZV55C10") (at 257.175 31.75 270) (unit 1)
-    (in_bom yes) (on_board yes) (dnp no) (fields_autoplaced)
-    (property "Reference" "D19" (at 260.35 30.48 90)
-      (effects (font (size 1.27 1.27)) (justify left))
-    )
-    (property "Value" "4.4-4.5 ZENER" (at 260.35 33.02 90)
-      (effects (font (size 1.27 1.27)) (justify left))
-    )
-    (property "Footprint" "Diode_SMD:D_SOD-123" (at 252.73 31.75 0)
-      (effects (font (size 1.27 1.27)) hide)
-    )
-    (property "Datasheet" "https://assets.nexperia.com/documents/data-sheet/BZV55_SER.pdf" (at 257.175 31.75 0)
+  (symbol (lib_id "Diode:BZV55C10") (at 281.94 31.75 270) (unit 1)
+    (in_bom yes) (on_board yes) (dnp no) (fields_autoplaced)
+    (property "Reference" "D19" (at 285.115 30.48 90)
+      (effects (font (size 1.27 1.27)) (justify left))
+    )
+    (property "Value" "4.4-4.5 ZENER" (at 285.115 33.02 90)
+      (effects (font (size 1.27 1.27)) (justify left))
+    )
+    (property "Footprint" "Diode_SMD:D_SOD-123" (at 277.495 31.75 0)
+      (effects (font (size 1.27 1.27)) hide)
+    )
+    (property "Datasheet" "https://assets.nexperia.com/documents/data-sheet/BZV55_SER.pdf" (at 281.94 31.75 0)
       (effects (font (size 1.27 1.27)) hide)
     )
@@
     )
   )
-  (symbol (lib_id "Connector:TestPoint") (at 260.985 27.94 0) (mirror y) (unit 1)
+  (symbol (lib_id "Connector:TestPoint") (at 285.75 27.94 0) (mirror y) (unit 1)
     (in_bom yes) (on_board yes) (dnp no)
-    (property "Reference" "SIM_PWR1" (at 267.843 25.4 0)
-      (effects (font (size 1.27 1.27)))
-    )
-    (property "Value" "TestPoint" (at 267.208 23.495 0)
-      (effects (font (size 1.27 1.27)))
-    )
-    (property "Footprint" "brilliant-kicad-library:TestPoint_Pad_D0.9mm" (at 255.905 27.94 0)
-      (effects (font (size 1.27 1.27)) hide)
-    )
-    (property "Datasheet" "~" (at 255.905 27.94 0)
+    (property "Reference" "SIM_PWR1" (at 292.608 25.4 0)
+      (effects (font (size 1.27 1.27)))
+    )
+    (property "Value" "TestPoint" (at 291.973 23.495 0)
+      (effects (font (size 1.27 1.27)))
+    )
+    (property "Footprint" "brilliant-kicad-library:TestPoint_Pad_D0.9mm" (at 280.67 27.94 0)
+      (effects (font (size 1.27 1.27)) hide)
+    )
+    (property "Datasheet" "~" (at 280.67 27.94 0)
       (effects (font (size 1.27 1.27)) hide)
     )
@@
     )
   )
-  (symbol (lib_id "power:GND") (at 257.175 45.72 0) (unit 1)
-    (in_bom yes) (on_board yes) (dnp no) (fields_autoplaced)
-    (property "Reference" "#PWR031" (at 257.175 52.07 0)
-      (effects (font (size 1.27 1.27)) hide)
-    )
-    (property "Value" "GND" (at 257.175 50.8 0)
-      (effects (font (size 1.27 1.27)))
-    )
-    (property "Footprint" "" (at 257.175 45.72 0)
-      (effects (font (size 1.27 1.27)) hide)
-    )
-    (property "Datasheet" "" (at 257.175 45.72 0)
+  (symbol (lib_id "power:GND") (at 281.94 45.72 0) (unit 1)
+    (in_bom yes) (on_board yes) (dnp no) (fields_autoplaced)
+    (property "Reference" "#PWR031" (at 281.94 52.07 0)
+      (effects (font (size 1.27 1.27)) hide)
+    )
+    (property "Value" "GND" (at 281.94 50.8 0)
+      (effects (font (size 1.27 1.27)))
+    )
+    (property "Footprint" "" (at 281.94 45.72 0)
+      (effects (font (size 1.27 1.27)) hide)
+    )
+    (property "Datasheet" "" (at 281.94 45.72 0)
       (effects (font (size 1.27 1.27)) hide)
     )
@@
     )
   )
-  (symbol (lib_id "Device:D_Schottky") (at 250.825 26.67 180) (unit 1)
-    (in_bom yes) (on_board yes) (dnp no) (fields_autoplaced)
-    (property "Reference" "D12" (at 251.1425 20.955 0)
-      (effects (font (size 1.27 1.27)))
-    )
-    (property "Value" "SS310" (at 251.1425 23.495 0)
-      (effects (font (size 1.27 1.27)))
-    )
-    (property "Footprint" "Diode_SMD:D_SMA" (at 250.825 26.67 0)
-      (effects (font (size 1.27 1.27)) hide)
-    )
-    (property "Datasheet" "~" (at 250.825 26.67 0)
+  (symbol (lib_id "Device:D_Schottky") (at 269.24 26.67 180) (unit 1)
+    (in_bom yes) (on_board yes) (dnp no) (fields_autoplaced)
+    (property "Reference" "D12" (at 269.5575 20.32 0)
+      (effects (font (size 1.27 1.27)))
+    )
+    (property "Value" "RS1K-E3/5ATSS310" (at 269.5575 22.86 0)
+      (effects (font (size 1.27 1.27)))
+    )
+    (property "Footprint" "Diode_SMD:D_SMA" (at 269.24 26.67 0)
+      (effects (font (size 1.27 1.27)) hide)
+    )
+    (property "Datasheet" "~" (at 269.24 26.67 0)
       (effects (font (size 1.27 1.27)) hide)
     )
@@
     )
   )
-  (symbol (lib_id "Device:R_US") (at 257.175 39.37 0) (unit 1)
-    (in_bom yes) (on_board yes) (dnp no) (fields_autoplaced)
-    (property "Reference" "R18" (at 259.715 38.735 0)
-      (effects (font (size 1.27 1.27)) (justify left))
-    )
-    (property "Value" "49.9R" (at 259.715 41.275 0)
-      (effects (font (size 1.27 1.27)) (justify left))
-    )
-    (property "Footprint" "Resistor_SMD:R_0402_1005Metric" (at 258.191 39.624 90)
-      (effects (font (size 1.27 1.27)) hide)
-    )
-    (property "Datasheet" "~" (at 257.175 39.37 0)
-      (effects (font (size 1.27 1.27)) hide)
-    )
+  (symbol (lib_id "Device:R_US") (at 281.94 39.37 0) (unit 1)
+    (in_bom yes) (on_board yes) (dnp no) (fields_autoplaced)
+    (property "Reference" "R18" (at 284.48 38.735 0)
+      (effects (font (size 1.27 1.27)) (justify left))
+    )
+    (property "Value" "49.9R" (at 284.48 41.275 0)
+      (effects (font (size 1.27 1.27)) (justify left))
+    )
+    (property "Footprint" "Resistor_SMD:R_0402_1005Metric" (at 282.956 39.624 90)
+      (effects (font (size 1.27 1.27)) hide)
+    )
+    (property "Datasheet" "~" (at 281.94 39.37 0)
+      (effects (font (size 1.27 1.27)) hide)
+    )
