File: SOURCE_FILES/BIM_PCB/STMFC8T6_MCU.kicad_sch (KiCad schematic)
At the start: 40 parts, among them J8 Conn_01x06, SW1 reset, U2 STM32F103C8Tx, Y1 8MHz, Y2 32.678KHz

Commit message: all items updated
Connections:
- net CAN_RX: now also U2.32 (PA11); no longer U2.22 (PB11)
- net CAN_TX: now also U2.33 (PA12); no longer U2.21 (PB10)
- net RS485_DI: now also U2.21 (PB10); no longer U2.32 (PA11)
- net RS485_RO: now also U2.22 (PB11); no longer U2.33 (PA12)
Changed lines of the file:
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@@
     (effects (font (size 1.27 1.27)) (justify left))
   )
-  (hierarchical_label "CAN_TX" (shape output) (at 108.585 118.745 180) (fields_autoplaced)
-    (effects (font (size 1.27 1.27)) (justify right))
+  (hierarchical_label "CAN_TX" (shape output) (at 177.165 123.825 0) (fields_autoplaced)
+    (effects (font (size 1.27 1.27)) (justify left))
   )
   (hierarchical_label "SW0" (shape input) (at 261.62 46.355 0) (fields_autoplaced)
@@
     (effects (font (size 1.27 1.27)) (justify left))
   )
-  (hierarchical_label "RS485_RO" (shape output) (at 177.165 123.825 0) (fields_autoplaced)
-    (effects (font (size 1.27 1.27) bold) (justify left))
+  (hierarchical_label "RS485_RO" (shape output) (at 108.585 121.285 180) (fields_autoplaced)
+    (effects (font (size 1.27 1.27) bold) (justify right))
   )
   (hierarchical_label "MUX_SEL_A" (shape output) (at 108.585 93.345 180) (fields_autoplaced)
@@
     (effects (font (size 1.27 1.27)) (justify left))
   )
-  (hierarchical_label "CAN_RX" (shape input) (at 108.585 121.285 180) (fields_autoplaced)
-    (effects (font (size 1.27 1.27)) (justify right))
+  (hierarchical_label "CAN_RX" (shape input) (at 177.165 121.285 0) (fields_autoplaced)
+    (effects (font (size 1.27 1.27)) (justify left))
   )
   (hierarchical_label "PWRKEY" (shape output) (at 108.0919 131.3658 180) (fields_autoplaced)
@@
     (effects (font (size 1.27 1.27)) (justify left))
   )
-  (hierarchical_label "RS485_DI" (shape input) (at 177.165 121.285 0) (fields_autoplaced)
-    (effects (font (size 1.27 1.27) bold) (justify left))
+  (hierarchical_label "RS485_DI" (shape input) (at 108.585 118.745 180) (fields_autoplaced)
+    (effects (font (size 1.27 1.27) bold) (justify right))
   )
   (hierarchical_label "SCL" (shape input) (at 108.585 108.585 180) (fields_autoplaced)
